File: 0_Hardware/1_Child_IO/2_8in8out/0_8in8out/v0.2.TYPED/8in8out.sch (KiCad schematic (older format))
At the start: 55 parts, among them IC1 ATTINY48-A, J1 RJ45, J2 RJ45, J3 CONN_6, K110 T771D10, K120 T771D10, K130 T771D10, K140 T771D10, K150 T771D10, K160 T771D10, K170 T771D10, K180 T771D10, P1 CONN_5, P100 CONN_2, P101 CONN_2, P102 CONN_2, P103 CONN_2, P105 CONN_2, P106 CONN_2, P110 CONN_2, P120 CONN_2, P130 CONN_2, P140 CONN_2, P150 CONN_2, P160 CONN_2, P170 CONN_2, P180 CONN_2, P2 CONN_5, P3 CONN_10X2, U1 7805, U2 ULN2803, U3 LTV847, U4 LTV847

Commit message: skilkscreen
Parts:
- removed U1: 7805, symbol 7805
- added U1: LM7805CT, TO-220, symbol LM7805CT
Connections:
- net +12V: now also U1.1 (IN)
- net +5V: now also U1.3 (OUT)
- net GND: now also U1.2 (GND)
Changed lines of the file:
@@
 Sheet 1 1
 Title "8in 8relays I2C board"
-Date "24 nov 2014"
+Date "28 nov 2014"
 Rev "V0.2"
 Comp "XPLDUINO project"
@@
 Text GLabel 18050 10250 0    60   Output ~ 0
 R7
-$Comp
-L 7805 U1
-U 1 1 516549E7
-P 12700 2550
-F 0 "U1" H 12850 2354 60  0000 C CNN
-F 1 "7805" H 12700 2750 60  0000 C CNN
-F 2 "" H 12700 2550 60  0000 C CNN
-F 3 "" H 12700 2550 60  0000 C CNN
-	1    12700 2550
-	1    0    0    -1
-$EndComp
 Wire Bus Line
 	12050 2000 13400 2000
@@
 Wire Wire Line
 	8500 4100 8500 4150
+$Comp
+L LM7805CT U1
+U 1 1 54789373
+P 12700 2550
+F 0 "U1" H 12500 2750 40  0000 C CNN
+F 1 "LM7805CT" H 12700 2750 40  0000 L CNN
+F 2 "TO-220" H 12700 2650 30  0000 C CIN
+F 3 "" H 12700 2550 60  0000 C CNN
+	1    12700 2550
+	1    0    0    -1
+$EndComp
 $EndSCHEMATC
